File: precharger.sch (KiCad schematic (older format))
At the start: 27 parts, among them J1 Conn_02x20_Odd_Even, Q1 2SC5200, Q2 2SC5200, Q3 MJL4302A, Q4 2SC5200, U1 ATmega328P-AU, U2 DCDC5Vout

Commit message: slower PWM needed because gate drive is lame
Parts:
- removed Q1: 2SC5200, Package_TO_SOT_SMD:SOT-89-3, symbol Transistor_BJT:BCX56
- removed R11: 36.5KΩ, symbol Device:R
- added C3, C4: 0.1μF, symbol Device:C
- added D5: 1N5817, symbol Device:D_Schottky
- added D6: POWER RED LED, symbol Device:LED
- added Q1: IPA60R400, symbol Device:Q_NMOS_SGD
- added Q5: 2N7000, symbol Device:Q_NMOS_SGD
- R1: value 150Ω -> 100KΩ
- R2: value 5Ω -> 360Ω
Connections:
- net labels added: IsenseGND, IsenseSig, IsenseVcc, VtwoVolts
- net labels removed: A3, Isignal
- wire segments 37 -> 46
Other:
- note added: "to enable Isense"
- moved on the sheet: U1

Commit message: add pullup resistor to DCDC, rm Q3 collector LED
Parts:
- removed D4: WHITE LED, symbol Device:LED
- added R11: 220KΩ, symbol Device:R
Connections:
- net labels added: DCDCinhibit
- net labels removed: DCDCenable
- wire segments 46 -> 51
Changed lines of the file:
@@
 $EndComp
 Wire Wire Line
-	9525 3700 9025 3700
+	9525 3700 9425 3700
 $Comp
 L Device:R R9
@@
 	6375 4725 6375 4525
 Text Label 6675 3175 0    50   ~ 0
-DCDCenable
+DCDCinhibit
 Connection ~ 9025 2900
 Wire Wire Line
@@
 Wire Wire Line
 	6375 4225 6375 4050
-Text Label 9825 3300 3    50   ~ 0
+Text Label 9825 3075 3    50   ~ 0
 yellow
 $Comp
@@
 	-1   0    0    -1
 $EndComp
-$Comp
-L Device:LED D4
-U 1 1 5CB1D027
-P 9825 3150
-F 0 "D4" V 9875 3350 50  0000 R CNN
-F 1 "WHITE LED" V 9775 3600 50  0000 R CNN
-F 2 "" H 9825 3150 50  0001 C CNN
-F 3 "~" H 9825 3150 50  0001 C CNN
-	1    9825 3150
-	0    -1   -1   0
-$EndComp
-Wire Wire Line
-	9825 3300 9825 3700
+Wire Wire Line
+	9825 3000 9825 3700
 Text Label 6675 3275 0    50   ~ 0
 green
@@
 	6525 2625 6525 2400
 Connection ~ 6225 2400
+$Comp
+L Device:R R11
+U 1 1 5CD69B8B
+P 6525 3175
+F 0 "R11" V 6318 3175 50  0000 C CNN
+F 1 "220KΩ" V 6409 3175 50  0000 C CNN
+F 2 "" V 6455 3175 50  0001 C CNN
+F 3 "~" H 6525 3175 50  0001 C CNN
+	1    6525 3175
+	0    1    1    0
+$EndComp
+Wire Wire Line
+	6375 3175 5925 3175
+Wire Wire Line
+	5925 3175 5925 4950
+Wire Wire Line
+	5925 4950 9425 4950
+Wire Wire Line
+	9425 4950 9425 3700
+Connection ~ 9425 3700
+Wire Wire Line
+	9425 3700 9025 3700
 $EndSCHEMATC
